File: edukate.kicad_pcb (KiCad board)
At the start: 2 copper layers, 93.4 x 152.7 mm, 76 parts, among them J1 Conn_LCD, J2 USB_OTG, Q1 C1815, Q2 C1815, SW1 KEY 1, SW10 KEY 6, SW11 KEY 9, SW12 KEY B, SW13 KEY C, SW14 KEY D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

Commit message: finished pcb layout
Parts:
- added G***: LOGO, MyKiCadLib:dolphin15x11, F.Cu at (91.5, 34.9)
- added REF**: ESD-Logo_8.9x8mm_SilkScreen, Symbol:ESD-Logo_8.9x8mm_SilkScreen, F.Cu at (101.4, 74.5)
- renumbered BT1 to BATT, POWER1 to BTN_POWER, JLINK1 to JLINK, RESET1 to RESET, SW_MNU1 to SW_MNU, UART1 to UART
Routing:
- net +3V3: track 0.00 -> 423.0 mm, vias 0 -> 15
- net +5V: track 0.00 -> 237.3 mm, vias 0 -> 7
- net /SW_MNU: track 0.00 -> 150.9 mm, vias 0 -> 4
- net Earth: track 10.8 -> 115.3 mm, vias 0 -> 197
- net /BOOT0: track 0.00 -> 103.3 mm, vias 0 -> 4
- net /LCD_RST: track 16.5 -> 78.5 mm, vias 0 -> 2
- net /BOOT1: track 0.00 -> 51.2 mm, vias 0 -> 2
- net /LCD_VOUT: track 0.00 -> 43.7 mm
- net -BATT: track 0.00 -> 24.9 mm
- net /LCD_RS: track 57.0 -> 78.1 mm
- net +BATT: track 0.00 -> 20.0 mm
- net Net-(U5-Pad1): track 0.00 -> 12.5 mm, vias 0 -> 2
- net /LCD_V0: track 0.00 -> 6.68 mm
- net Net-(D1-Pad2): track 0.00 -> 4.41 mm
- net Net-(R10-Pad1): track 0.00 -> 4.33 mm
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- added copper zone on F.Cu, net +3V3
- added copper zone on F.Cu, net +5V
- added copper zone on B.Cu, net +BATT
- added copper zone on F.Cu, net +BATT
- added copper zone on F.Cu, net +VSW
- added copper zone on F.Cu, net -BATT
- added copper zone on B.Cu, net Earth
- added copper zone on F.Cu, net Earth
- added copper zone on F.Cu, net Net-(D1-Pad2)
- added copper zone on F.Cu, net Net-(L2-Pad1)
Other:
- board text added: "+"
- board text added: "+3V3"
- board text added: "+5V"
- board text added: "-"
- board text added: "0"
- board text added: "1"
- board text added: "2"
- board text added: "3"
- board text added: "4"
- board text added: "5"
- board text added: "6"
- board text added: "7"
- board text added: "8"
- board text added: "9"
- board text added: "A"
- board text added: "B"
- board text added: "C"
- board text added: "D"
- board text added: "E"
- board text added: "EDUKATE - CHIP 8 EMULATOR"
- board text added: "F"
- board text added: "GND"
- board text added: "RX"
- board text added: "SWDCLK"
- board text added: "SWDIO"
- board text added: "TX"
